Commit message: Change project names to omniwheel_base

File: urdf/description.urdf (robot description, URDF)
Before this commit: robot open_base, 29 links, 28 joints
Links:
- link back_rim_link: geometry collision mesh filename=package://omniwheel_base/mesh/rim.stl; visual mesh filename=package://omniwheel_base/mesh/rim.stl
- link back_roller_e_link: geometry collision mesh filename=package://omniwheel_base/mesh/roller.stl; visual mesh filename=package://omniwheel_base/mesh/roller.stl
- link back_roller_n_link: geometry collision mesh filename=package://omniwheel_base/mesh/roller.stl; visual mesh filename=package://omniwheel_base/mesh/roller.stl
- link back_roller_ne_link: geometry collision mesh filename=package://omniwheel_base/mesh/roller.stl; visual mesh filename=package://omniwheel_base/mesh/roller.stl
- link back_roller_nw_link: geometry collision mesh filename=package://omniwheel_base/mesh/roller.stl; visual mesh filename=package://omniwheel_base/mesh/roller.stl
- link back_roller_s_link: geometry collision mesh filename=package://omniwheel_base/mesh/roller.stl; visual mesh filename=package://omniwheel_base/mesh/roller.stl
- link back_roller_se_link: geometry collision mesh filename=package://omniwheel_base/mesh/roller.stl; visual mesh filename=package://omniwheel_base/mesh/roller.stl
- link back_roller_sw_link: geometry collision mesh filename=package://omniwheel_base/mesh/roller.stl; visual mesh filename=package://omniwheel_base/mesh/roller.stl
- link back_roller_w_link: geometry collision mesh filename=package://omniwheel_base/mesh/roller.stl; visual mesh filename=package://omniwheel_base/mesh/roller.stl
- link base_link: geometry collision mesh filename=package://omniwheel_base/mesh/base.stl; visual mesh filename=package://omniwheel_base/mesh/base.stl
- link left_rim_link: geometry collision mesh filename=package://omniwheel_base/mesh/rim.stl; visual mesh filename=package://omniwheel_base/mesh/rim.stl
- link left_roller_e_link: geometry collision mesh filename=package://omniwheel_base/mesh/roller.stl; visual mesh filename=package://omniwheel_base/mesh/roller.stl
- link left_roller_n_link: geometry collision mesh filename=package://omniwheel_base/mesh/roller.stl; visual mesh filename=package://omniwheel_base/mesh/roller.stl
- link left_roller_ne_link: geometry collision mesh filename=package://omniwheel_base/mesh/roller.stl; visual mesh filename=package://omniwheel_base/mesh/roller.stl
- link left_roller_nw_link: geometry collision mesh filename=package://omniwheel_base/mesh/roller.stl; visual mesh filename=package://omniwheel_base/mesh/roller.stl
- link left_roller_s_link: geometry collision mesh filename=package://omniwheel_base/mesh/roller.stl; visual mesh filename=package://omniwheel_base/mesh/roller.stl
- link left_roller_se_link: geometry collision mesh filename=package://omniwheel_base/mesh/roller.stl; visual mesh filename=package://omniwheel_base/mesh/roller.stl
- link left_roller_sw_link: geometry collision mesh filename=package://omniwheel_base/mesh/roller.stl; visual mesh filename=package://omniwheel_base/mesh/roller.stl
- link left_roller_w_link: geometry collision mesh filename=package://omniwheel_base/mesh/roller.stl; visual mesh filename=package://omniwheel_base/mesh/roller.stl
- link right_rim_link: geometry collision mesh filename=package://omniwheel_base/mesh/rim.stl; visual mesh filename=package://omniwheel_base/mesh/rim.stl
- link right_roller_e_link: geometry collision mesh filename=package://omniwheel_base/mesh/roller.stl; visual mesh filename=package://omniwheel_base/mesh/roller.stl
- link right_roller_n_link: geometry collision mesh filename=package://omniwheel_base/mesh/roller.stl; visual mesh filename=package://omniwheel_base/mesh/roller.stl
- link right_roller_ne_link: geometry collision mesh filename=package://omniwheel_base/mesh/roller.stl; visual mesh filename=package://omniwheel_base/mesh/roller.stl
- link right_roller_nw_link: geometry collision mesh filename=package://omniwheel_base/mesh/roller.stl; visual mesh filename=package://omniwheel_base/mesh/roller.stl
- link right_roller_s_link: geometry collision mesh filename=package://omniwheel_base/mesh/roller.stl; visual mesh filename=package://omniwheel_base/mesh/roller.stl
- link right_roller_se_link: geometry collision mesh filename=package://omniwheel_base/mesh/roller.stl; visual mesh filename=package://omniwheel_base/mesh/roller.stl
- link right_roller_sw_link: geometry collision mesh filename=package://omniwheel_base/mesh/roller.stl; visual mesh filename=package://omniwheel_base/mesh/roller.stl
- link right_roller_w_link: geometry collision mesh filename=package://omniwheel_base/mesh/roller.stl; visual mesh filename=package://omniwheel_base/mesh/roller.stl

File: xacro/main.urdf.xacro (robot description, xacro)
@@ -2,7 +2,7 @@
 <robot
 	xmlns:xacro="http://www.ros.org/wiki/xacro"
-	name="open_base"
+	name="omniwheel_base"
 >
-	<xacro:include filename="$(find open_base)/xacro/rim.urdf.xacro"/>
+	<xacro:include filename="$(find omniwheel_base)/xacro/rim.urdf.xacro"/>
 	<link name="origin_link"/>
 	<link name="base_link">
@@ -20,5 +20,5 @@
 	<visual>
 		<geometry>
-			<mesh filename="package://open_base/mesh/base.stl"/>
+			<mesh filename="package://omniwheel_base/mesh/base.stl"/>
 		</geometry>
 		<material name="base_material">
@@ -28,5 +28,5 @@
 	<collision>
 		<geometry>
-			<mesh filename="package://open_base/mesh/base.stl"/>
+			<mesh filename="package://omniwheel_base/mesh/base.stl"/>
 		</geometry>
 	</collision>
@@ -62,5 +62,5 @@
 	<gazebo>
 		<plugin name="gazebo_ros_control" filename="libgazebo_ros_control.so">
-			<robotNamespace>/open_base</robotNamespace>
+			<robotNamespace>/omniwheel_base</robotNamespace>
 		</plugin>
 	</gazebo>

File: xacro/rim.urdf.xacro (robot description, xacro)
@@ -1,5 +1,5 @@
 <?xml version="1.0" ?>
 <robot xmlns:xacro="http://www.ros.org/wiki/xacro">
-	<xacro:include filename="$(find open_base)/xacro/roller.urdf.xacro"/>
+	<xacro:include filename="$(find omniwheel_base)/xacro/roller.urdf.xacro"/>
 	<xacro:macro
 		name="rim_macro"
@@ -21,5 +21,5 @@
 			<visual>
 				<geometry>
-					<mesh filename="package://open_base/mesh/rim.stl"/>
+					<mesh filename="package://omniwheel_base/mesh/rim.stl"/>
 				</geometry>
 				<material name="rim_${name}_material">
@@ -29,5 +29,5 @@
 			<collision>
 				<geometry>
-					<mesh filename="package://open_base/mesh/rim.stl"/>
+					<mesh filename="package://omniwheel_base/mesh/rim.stl"/>
 				</geometry>
 			</collision>

File: xacro/roller.urdf.xacro (robot description, xacro)
@@ -19,5 +19,5 @@
 			<visual>
 				<geometry>
-					<mesh filename="package://open_base/mesh/roller.stl"/>
+					<mesh filename="package://omniwheel_base/mesh/roller.stl"/>
 				</geometry>
 				<material name="roller_material">
@@ -27,5 +27,5 @@
 			<collision>
 				<geometry>
-					<mesh filename="package://open_base/mesh/roller.stl"/>
+					<mesh filename="package://omniwheel_base/mesh/roller.stl"/>
 				</geometry>
 			</collision>
