Commit message: renaming & cleaning

File: urdf/gambot.urdf (robot description, URDF)
Before this commit: robot gambot, 29 links, 28 joints
Links:
- link back_rim_link: geometry collision mesh filename=package://gambot_base/mesh/rim.stl; visual mesh filename=package://gambot_base/mesh/rim.stl
- link back_roller_e_link: geometry collision mesh filename=package://gambot_base/mesh/roller.stl; visual mesh filename=package://gambot_base/mesh/roller.stl
- link back_roller_n_link: geometry collision mesh filename=package://gambot_base/mesh/roller.stl; visual mesh filename=package://gambot_base/mesh/roller.stl
- link back_roller_ne_link: geometry collision mesh filename=package://gambot_base/mesh/roller.stl; visual mesh filename=package://gambot_base/mesh/roller.stl
- link back_roller_nw_link: geometry collision mesh filename=package://gambot_base/mesh/roller.stl; visual mesh filename=package://gambot_base/mesh/roller.stl
- link back_roller_s_link: geometry collision mesh filename=package://gambot_base/mesh/roller.stl; visual mesh filename=package://gambot_base/mesh/roller.stl
- link back_roller_se_link: geometry collision mesh filename=package://gambot_base/mesh/roller.stl; visual mesh filename=package://gambot_base/mesh/roller.stl
- link back_roller_sw_link: geometry collision mesh filename=package://gambot_base/mesh/roller.stl; visual mesh filename=package://gambot_base/mesh/roller.stl
- link back_roller_w_link: geometry collision mesh filename=package://gambot_base/mesh/roller.stl; visual mesh filename=package://gambot_base/mesh/roller.stl
- link base_link: geometry collision mesh filename=package://gambot_base/mesh/base.stl; visual mesh filename=package://gambot_base/mesh/base.stl
- link left_rim_link: geometry collision mesh filename=package://gambot_base/mesh/rim.stl; visual mesh filename=package://gambot_base/mesh/rim.stl
- link left_roller_e_link: geometry collision mesh filename=package://gambot_base/mesh/roller.stl; visual mesh filename=package://gambot_base/mesh/roller.stl
- link left_roller_n_link: geometry collision mesh filename=package://gambot_base/mesh/roller.stl; visual mesh filename=package://gambot_base/mesh/roller.stl
- link left_roller_ne_link: geometry collision mesh filename=package://gambot_base/mesh/roller.stl; visual mesh filename=package://gambot_base/mesh/roller.stl
- link left_roller_nw_link: geometry collision mesh filename=package://gambot_base/mesh/roller.stl; visual mesh filename=package://gambot_base/mesh/roller.stl
- link left_roller_s_link: geometry collision mesh filename=package://gambot_base/mesh/roller.stl; visual mesh filename=package://gambot_base/mesh/roller.stl
- link left_roller_se_link: geometry collision mesh filename=package://gambot_base/mesh/roller.stl; visual mesh filename=package://gambot_base/mesh/roller.stl
- link left_roller_sw_link: geometry collision mesh filename=package://gambot_base/mesh/roller.stl; visual mesh filename=package://gambot_base/mesh/roller.stl
- link left_roller_w_link: geometry collision mesh filename=package://gambot_base/mesh/roller.stl; visual mesh filename=package://gambot_base/mesh/roller.stl
- link right_rim_link: geometry collision mesh filename=package://gambot_base/mesh/rim.stl; visual mesh filename=package://gambot_base/mesh/rim.stl
- link right_roller_e_link: geometry collision mesh filename=package://gambot_base/mesh/roller.stl; visual mesh filename=package://gambot_base/mesh/roller.stl
- link right_roller_n_link: geometry collision mesh filename=package://gambot_base/mesh/roller.stl; visual mesh filename=package://gambot_base/mesh/roller.stl
- link right_roller_ne_link: geometry collision mesh filename=package://gambot_base/mesh/roller.stl; visual mesh filename=package://gambot_base/mesh/roller.stl
- link right_roller_nw_link: geometry collision mesh filename=package://gambot_base/mesh/roller.stl; visual mesh filename=package://gambot_base/mesh/roller.stl
- link right_roller_s_link: geometry collision mesh filename=package://gambot_base/mesh/roller.stl; visual mesh filename=package://gambot_base/mesh/roller.stl
- link right_roller_se_link: geometry collision mesh filename=package://gambot_base/mesh/roller.stl; visual mesh filename=package://gambot_base/mesh/roller.stl
- link right_roller_sw_link: geometry collision mesh filename=package://gambot_base/mesh/roller.stl; visual mesh filename=package://gambot_base/mesh/roller.stl
- link right_roller_w_link: geometry collision mesh filename=package://gambot_base/mesh/roller.stl; visual mesh filename=package://gambot_base/mesh/roller.stl

Commit message: Change base_link's parent to base_footprint

File: urdf/gambot.urdf (robot description, URDF)
Before this commit: robot gambot, 29 links, 28 joints
Links:
- removed link origin_link
- added link base_footprint
Joints:
- joint origin_joint: parent origin_link -> base_footprint
